File: hw/ESP-Breakout.kicad_pcb (KiCad board)
At the start: 2 copper layers, 50.8 x 20.3 mm, 17 parts, among them M1 ESP-07, P1 FTDI BASIC, P2 CONN_01X11, P3 CONN_01X11, Q1 BSS138, Q2 BSS138, SW1 SW_PUSH, U1 1117-3.3

Commit message: Upgraded to KiCad 7.0
The schematic symbols have been manually paired with KiCad's standard ones.
The footprints on the PCB have not been changed to preserve the layout.
Other:
- net class Default removed
